Commit message: Add standing pose and stabilization changes

File: g1_control/g1_23dof_control.urdf (robot description, URDF)
Before this commit: robot g1_23dof, 33 links, 32 joints
Links:
- link head_link: geometry collision mesh filename=file:///home/pcmc/unitree_ws/src/g1_description/meshes/head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; visual box 
Joints:
- joint left_elbow_joint: axis 0 1 0 -> (none); limit lower=-1.0472 upper=2.0944 effort=25 velocity=37 -> (none); type revolute -> fixed
- joint left_shoulder_pitch_joint: axis 0 1 0 -> (none); limit lower=-3.0892 upper=2.6704 effort=25 velocity=37 -> (none); type revolute -> fixed
- joint left_shoulder_roll_joint: axis 1 0 0 -> (none); limit lower=-1.5882 upper=2.2515 effort=25 velocity=37 -> (none); type revolute -> fixed
- joint left_shoulder_yaw_joint: axis 0 0 1 -> (none); limit lower=-2.618 upper=2.618 effort=25 velocity=37 -> (none); type revolute -> fixed
- joint left_wrist_roll_joint: axis 1 0 0 -> (none); limit lower=-1.972222054 upper=1.972222054 effort=25 velocity=37 -> (none); type revolute -> fixed
- joint right_elbow_joint: axis 0 1 0 -> (none); limit lower=-1.0472 upper=2.0944 effort=25 velocity=37 -> (none); type revolute -> fixed
- joint right_shoulder_pitch_joint: axis 0 1 0 -> (none); limit lower=-3.0892 upper=2.6704 effort=25 velocity=37 -> (none); type revolute -> fixed
- joint right_shoulder_roll_joint: axis 1 0 0 -> (none); limit lower=-2.2515 upper=1.5882 effort=25 velocity=37 -> (none); type revolute -> fixed
- joint right_shoulder_yaw_joint: axis 0 0 1 -> (none); limit lower=-2.618 upper=2.618 effort=25 velocity=37 -> (none); type revolute -> fixed
- joint right_wrist_roll_joint: axis 1 0 0 -> (none); limit lower=-1.972222054 upper=1.972222054 effort=25 velocity=37 -> (none); type revolute -> fixed
